File: PCB/power.kicad_sch (KiCad schematic)
At the start: 11 parts, among them J2 5V, U4 AP2112K-3.3, U5 MAX40200AUK

Commit message: Generate project from template
Other:
- title: template_pretty_name -> EOS Homework Board
Changed lines of the file:
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@@
 	(paper "A4")
 	(title_block
-		(title "template_pretty_name")
+		(title "EOS Homework Board")
 	)
 	(text "5V -> 3.3V LDO"
